Commit message: fix mapping and navigation nodes

File: urdf/wheeltec/sensor.xacro (robot description, xacro)
@@ -3,5 +3,5 @@
   <!-- laser -->
   <joint name="$(arg namespace)/laser_joint" type="fixed">
-    <origin xyz="0.03 0.00 0.18" rpy="0 0 0" />
+    <origin xyz="0.03 0.00 0.18" rpy="0 0 3.14" />
     <parent link="$(arg namespace)/base_link" />
     <child link="$(arg namespace)/laser_link" />
